File: handheld/handmade01/main.sch (KiCad schematic (older format))
At the start: 75 parts, among them CON1 MicroSD, CON2 MicroSD, J1 JACK_TRS_6PINS, P1 VOLUMN, P4 USB_OTG, P6 UART_DEBUG, Q1 1AM, SW1 Power, SW10 R, SW11 A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

Commit message: updated core library
Parts:
- removed R10, R11, R12, R13, R14, R15, R16, R17, R18, R19, R21, R23, R24, R25, R26, R27, R28, R29, R30, R5, R6, R7, R8, R9: 4.7K, symbol R
- removed SW10: R, symbol SW_Push
- removed SW11: A, symbol SW_Push
- removed SW12: B, symbol SW_Push
- removed SW13: X, symbol SW_Push
- removed SW14: Y, symbol SW_Push
- removed SW3: UP, symbol SW_Push
- removed SW4: Down, symbol SW_Push
- removed SW5: Left, symbol SW_Push
- removed SW6: Right, symbol SW_Push
- removed SW7: Select, symbol SW_Push
- removed SW8: Start, symbol SW_Push
- removed SW9: L, symbol SW_Push
- added RN1: R_Network10, Resistors_ThroughHole:Resistor_Array_SIP11, symbol R_Network10
- added RN2, RN3: R_Network07, Resistors_ThroughHole:Resistor_Array_SIP8, symbol R_Network07
- added U10: NDSL_LR, symbol NDSL_LR
- added U?: NDSL_4BTN, symbol NDSL_4BTN
- added U?: NDSL_DPad, symbol NDSL_DPad
- added U?: NDSL_SS, symbol NDSL_SS
- C1, C10, C11, C12, C2, C3, C4, C5, C6, C7, C8, C9: symbol C -> C-RESCUE-main
- R1, R2, R20, R22, R3, R4: symbol R -> R-RESCUE-main
- SW1, SW2: symbol SW_Push -> SW_PUSH
- U6, U7: symbol CONN-38PIN -> Conn-38Pin
- U8, U9: symbol CONN-32PIN -> Conn-32Pin
Connections:
- wire segments 40 -> 22
Other:
- note removed: "Handmade01"
- moved on the sheet: BAT1, C11, C12, CON1, CON2, J1, LS1, LS2, P1, P4, P6, Q1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
