File: core/common/main.kicad_pcb (KiCad board)
At the start: 2 copper layers, 99.1 x 49.8 mm, 7 parts, among them P1 CONN_01X05, P2 CONN_01X03, P3 CONN_01X02, P4 CONN_01X02, U1 NDSL_DPad, U2 NDSL_SS, U3 N900_Keyboard

Commit message: updated n900 and blackberry q30 sch & pcb
Parts:
- added P5: CONN_01X28, Housings_SOIC:SOIC-28W_7.5x17.9mm_Pitch1.27mm, B.Cu at (121.2, 121.7)
- added P7: CONN_01X28, steward:MyFT_BM14B(0.8)-24DS-0.4V(51), F.Cu at (120.9, 121.9)
- added P8: CONN_01X28, Housings_SOIC:SOIC-28W_7.5x17.9mm_Pitch1.27mm, F.Cu at (121.2, 121.7)
- added U4: N900_Keyboard, steward:MyFT_N900_Keyboard_Pinout, F.Cu at (102.6, 145.5)
Connections:
- U3 pad 1: Net-(U3-Pad1) -> K1
- U3 pad 10: Net-(U3-Pad10) -> K10
- U3 pad 11: Net-(U3-Pad11) -> K11
- U3 pad 12: Net-(U3-Pad12) -> K12
- U3 pad 13: Net-(U3-Pad13) -> K13
- U3 pad 14: Net-(U3-Pad14) -> K14
- U3 pad 15: Net-(U3-Pad15) -> K15
- U3 pad 16: Net-(U3-Pad16) -> K16
- U3 pad 2: Net-(U3-Pad2) -> K2
- U3 pad 3: Net-(U3-Pad3) -> K3
- U3 pad 4: Net-(U3-Pad4) -> K4
- U3 pad 5: Net-(U3-Pad5) -> K5
- U3 pad 6: Net-(U3-Pad6) -> K6
- U3 pad 7: Net-(U3-Pad7) -> K7
- U3 pad 8: Net-(U3-Pad8) -> K8
- U3 pad 9: Net-(U3-Pad9) -> K9
Routing:
- net Net-(U3-Pad16): track 85.3 -> 0.00 mm
- net Net-(U3-Pad14): track 85.3 -> 0.00 mm
- net K16: track 0.00 -> 85.3 mm, vias 0 -> 1
- net K14: track 0.00 -> 85.3 mm
- net Net-(U3-Pad15): track 85.3 -> 0.00 mm
- net K15: track 0.00 -> 85.3 mm
- net Net-(U3-Pad11): track 12.1 -> 0.00 mm, vias 5 -> 0
- net K11: track 0.00 -> 12.1 mm, vias 0 -> 5
- net Net-(U3-Pad9): track 12.1 -> 0.00 mm, vias 4 -> 0
- net Net-(U3-Pad8): track 12.1 -> 0.00 mm, vias 4 -> 0
- net Net-(U3-Pad7): track 12.1 -> 0.00 mm, vias 4 -> 0
- net Net-(U3-Pad6): track 12.1 -> 0.00 mm, vias 4 -> 0
- net Net-(U3-Pad5): track 12.1 -> 0.00 mm, vias 4 -> 0
- net Net-(U3-Pad4): track 12.1 -> 0.00 mm, vias 4 -> 0
- net Net-(U3-Pad3): track 12.1 -> 0.00 mm, vias 4 -> 0
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Other:
- outline, holes or cut-outs redrawn

Commit message: updated n900 pcb
Parts:
- U4: moved to B.Cu
- moved U4 6.55 mm to (109.2, 145.5), turned to 180 degrees
Connections:
- U4 pad 1: K1 -> K13
- U4 pad 10: K10 -> K4
- U4 pad 11: K11 -> K3
- U4 pad 12: K12 -> K2
- U4 pad 13: K13 -> K1
- U4 pad 2: K2 -> K12
- U4 pad 3: K3 -> K11
- U4 pad 4: K4 -> K10
- U4 pad 5: K5 -> K9
- U4 pad 6: K6 -> K8
- U4 pad 8: K8 -> K6
- U4 pad 9: K9 -> K5
Routing:
- net K16: track 85.3 -> 87.6 mm
- net K14: track 85.3 -> 87.6 mm, vias 0 -> 1
- net K15: track 85.3 -> 87.6 mm, vias 0 -> 1
Other:
- outline, holes or cut-outs redrawn
